File: SPECTRE_V0.5.3/Speeduino_base.sch (KiCad schematic (older format))
At the start: 197 parts, among them J1 Conn_01x06_Male, J2 Conn_02x04_Odd_Even, J3 ProtoArea, Q1 AO3400, Q10 BSP78, Q11 BSP78, Q12 AO3400, Q13 BSP78, Q14 BSP78, Q15 BSP78, Q16 BSP78, Q17 BSP78, Q18 BSP78, Q19 BSP78, Q20 BSP78, Q21 BSP78, Q6 AO3400, Q7 AO3400, U1 MAX9926UAEE+, U10 MIC4427, U2 LM78M05_TO220, U3 TL431DBZ, U4 molex_48pin, U5 TJA1050, U6 MAX3232, U7 MIC4427, U8 MIC4427, U9 MIC4427

Commit message: Increased VBAT width
Parts:
- removed unit 4 of RN1
- removed unit 4 of RN2
- removed U4: molex_48pin, Speeduino_base:Molex_48, symbol Speeduino_base-rescue:molex_48pin-molex_48pin
- added unit 3 of RN1
- added unit 3 of RN2
- added U4: molex_48pin, Speeduino_base:Molex_48, symbol speeduino_lib:molex_48pin
Other:
- moved on the sheet: JP15, JP16, JP18, JP5, JP6, JP7, JP8
