File: SPECTRE_V0.5.4/Speeduino_base.kicad_pcb (KiCad board)
At the start: 2 copper layers, 100 x 93 mm, 197 parts, among them J1 Conn_01x06_Male, J2 Conn_02x04_Odd_Even, J3 ProtoArea, Q1 AO3400, Q10 BSP78, Q11 BSP78, Q12 AO3400, Q13 BSP78, Q14 BSP78, Q15 BSP78, Q16 BSP78, Q17 BSP78, Q18 BSP78, Q19 BSP78, Q20 BSP78, Q21 BSP78, Q6 AO3400, Q7 AO3400, U1 MAX9926UAEE+, U10 MIC4427, U2 LM78M05_TO220, U3 TL431DBZ, U4 molex_48pin, U5 TJA1050, U6 MAX3232, U7 MIC4427, U8 MIC4427, U9 MIC4427

Commit message: Update Speeduino_base.kicad_pcb
Parts:
- moved F2 3.28 mm to (179.6, 69.1), turned to 270 degrees
- moved D31 0.57 mm to (161.0, 65.0)
- moved D32 0.57 mm to (156.7, 65.0)
- turned C15 to 0 degrees
Routing:
- net 5V: track 389.1 -> 365.2 mm, vias 6 -> 8
- net INJ8-OUT: track 42.5 -> 56.9 mm, vias 1 -> 3
- net Net-(D36-Pad1): track 37.8 -> 42.6 mm, vias 1 -> 5
- net INJ3-OUT: track 56.0 -> 60.5 mm, vias 3 -> 7
- net IDLE1-OUT: track 24.1 -> 27.1 mm, vias 1 -> 3
- net INJ2-OUT: track 37.1 -> 40.0 mm, vias 1 -> 5
- net V_IDLE: track 16.7 -> 14.1 mm
- net VBAT: track 320.1 -> 322.5 mm, vias 13 -> 15
- net PWR_GND: track 160.5 -> 158.5 mm, vias 145 -> 150
- net Net-(D39-Pad1): track 37.6 -> 35.7 mm, vias 1 -> 3
- net Spare_2-Out: track 13.0 -> 11.4 mm, vias 2 -> 0
- net INJ6-OUT: track 29.8 -> 31.3 mm, vias 1 -> 3
- net BOOST-OUT: track 21.9 -> 23.4 mm, vias 0 -> 2
- net IDLE2-OUT: track 17.9 -> 19.3 mm, vias 1 -> 3
- net Net-(D43-Pad1): track 48.0 -> 46.7 mm, vias 1 -> 3
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
Commit message: Update Speeduino_base.kicad_pcb
Routing:
- net PWR_GND: vias 150 -> 153
- net GND: vias 121 -> 133
Other:
- board text added: "SPECTRE STM32F4 Speeduino compatible V0.5.4"
- board text removed: "SPECTRE STM32F4 Speeduino compatible V0.5.3"

Commit message: Minor changes
Routing:
- net INJ5-OUT: track 31.7 -> 32.2 mm
- net VBAT: vias 15 -> 16
- net PWR_GND: vias 153 -> 154
